File: lora_nodemcu.sch (KiCad schematic (older format))
At the start: 3 parts, among them U1 RFM95, U2 NodeMCU_Amica_R2

Commit message: starting on board layout
Parts:
- added R1, R2, R3: R, symbol R
Changed lines of the file:
@@
 L NodeMCU_Amica_R2 U2
 U 1 1 59CB0B60
-P 7250 3250
-F 0 "U2" H 7250 4050 50  0000 C CNN
-F 1 "NodeMCU_Amica_R2" H 7250 2400 50  0000 C CNN
-F 2 "" H 7500 3250 50  0000 C CNN
-F 3 "" H 7500 3250 50  0000 C CNN
-	1    7250 3250
+P 7850 3100
+F 0 "U2" H 7850 3900 50  0000 C CNN
+F 1 "NodeMCU_Amica_R2" H 7850 2250 50  0000 C CNN
+F 2 "" H 8100 3100 50  0000 C CNN
+F 3 "" H 8100 3100 50  0000 C CNN
+	1    7850 3100
 	1    0    0    -1
 $EndComp
@@
 	4500 3400 4350 3400
 $Comp
-L GND #PWR3
+L GND #PWR01
 U 1 1 59CB0D77
 P 5800 3650
-F 0 "#PWR3" H 5800 3400 50  0001 C CNN
+F 0 "#PWR01" H 5800 3400 50  0001 C CNN
 F 1 "GND" H 5800 3500 50  0000 C CNN
 F 2 "" H 5800 3650 50  0001 C CNN
@@
 $EndComp
 $Comp
-L GND #PWR2
+L GND #PWR02
 U 1 1 59CB0DA4
 P 5700 2600
-F 0 "#PWR2" H 5700 2350 50  0001 C CNN
+F 0 "#PWR02" H 5700 2350 50  0001 C CNN
 F 1 "GND" H 5700 2450 50  0000 C CNN
 F 2 "" H 5700 2600 50  0001 C CNN
@@
 	5800 3500 5800 3650
 Wire Wire Line
-	6800 3350 6400 3350
-Wire Wire Line
-	6400 3350 6400 3200
-Wire Wire Line
-	6400 3200 5700 3200
+	6700 3200 7400 3200
 $Comp
-L +3.3V #PWR1
+L +3.3V #PWR03
 U 1 1 59CB1055
 P 4250 3100
-F 0 "#PWR1" H 4250 2950 50  0001 C CNN
+F 0 "#PWR03" H 4250 2950 50  0001 C CNN
 F 1 "+3.3V" H 4250 3240 50  0000 C CNN
 F 2 "" H 4250 3100 50  0001 C CNN
@@
 	4350 3400 4350 3950
 $Comp
-L GND #PWR5
+L GND #PWR04
 U 1 1 59CB1286
-P 6550 3850
-F 0 "#PWR5" H 6550 3600 50  0001 C CNN
-F 1 "GND" H 6550 3700 50  0000 C CNN
-F 2 "" H 6550 3850 50  0001 C CNN
-F 3 "" H 6550 3850 50  0001 C CNN
-	1    6550 3850
+P 7150 3700
+F 0 "#PWR04" H 7150 3450 50  0001 C CNN
+F 1 "GND" H 7150 3550 50  0000 C CNN
+F 2 "" H 7150 3700 50  0001 C CNN
+F 3 "" H 7150 3700 50  0001 C CNN
+	1    7150 3700
 	0    1    1    0
 $EndComp
 Wire Wire Line
-	6800 3850 6550 3850
+	7400 3700 7150 3700
 $Comp
-L +3.3V #PWR6
+L +3.3V #PWR05
 U 1 1 59CB12BC
-P 7900 3950
-F 0 "#PWR6" H 7900 3800 50  0001 C CNN
-F 1 "+3.3V" H 7900 4090 50  0000 C CNN
-F 2 "" H 7900 3950 50  0001 C CNN
-F 3 "" H 7900 3950 50  0001 C CNN
-	1    7900 3950
+P 8500 3800
+F 0 "#PWR05" H 8500 3650 50  0001 C CNN
+F 1 "+3.3V" H 8500 3940 50  0000 C CNN
+F 2 "" H 8500 3800 50  0001 C CNN
+F 3 "" H 8500 3800 50  0001 C CNN
+	1    8500 3800
 	0    1    1    0
 $EndComp
 Wire Wire Line
-	7700 3950 7900 3950
-Wire Wire Line
-	6800 3050 6150 3050
-Wire Wire Line
-	6150 3050 6150 3300
-Wire Wire Line
-	6150 3300 5700 3300
-Text Label 6350 3050 0    60   ~ 0
+	8300 3800 8500 3800
+Text Label 7100 2900 0    60   ~ 0
 MOSI
 Wire Wire Line
-	6800 3250 6300 3250
-Wire Wire Line
-	6300 3250 6300 3400
-Wire Wire Line
-	6300 3400 5700 3400
-Text Label 6500 3250 0    60   ~ 0
+	7400 3100 6900 3100
+Text Label 7100 3100 0    60   ~ 0
 MISO
 $Comp
-L +3.3V #PWR4
+L +3.3V #PWR06
 U 1 1 59CB148A
-P 6500 3550
-F 0 "#PWR4" H 6500 3400 50  0001 C CNN
-F 1 "+3.3V" H 6500 3690 50  0000 C CNN
-F 2 "" H 6500 3550 50  0001 C CNN
-F 3 "" H 6500 3550 50  0001 C CNN
-	1    6500 3550
+P 7100 3400
+F 0 "#PWR06" H 7100 3250 50  0001 C CNN
+F 1 "+3.3V" H 7100 3540 50  0000 C CNN
+F 2 "" H 7100 3400 50  0001 C CNN
+F 3 "" H 7100 3400 50  0001 C CNN
+	1    7100 3400
 	0    -1   -1   0
 $EndComp
 Wire Wire Line
-	6800 3550 6500 3550
+	7400 3400 7100 3400
+Text Label 7150 3000 0    60   ~ 0
+CS
+$Comp
+L R R3
+U 1 1 59CC447A
+P 6750 2900
+F 0 "R3" V 6830 2900 50  0000 C CNN
+F 1 "R" V 6750 2900 50  0000 C CNN
+F 2 "" V 6680 2900 50  0001 C CNN
+F 3 "" H 6750 2900 50  0001 C CNN
+	1    6750 2900
+	0    1    1    0
+$EndComp
 Wire Wire Line
-	6800 3150 6000 3150
+	7150 1700 3300 1700
 Wire Wire Line
-	6000 3150 6000 3100
+	3300 1700 3300 550
 Wire Wire Line
-	6000 3100 5700 3100
-Text Label 6550 3150 0    60   ~ 0
-CS
+	7400 2900 6900 2900
+Wire Wire Line
+	5700 3300 5900 3300
+Wire Wire Line
+	5700 3200 6400 3200
+Wire Wire Line
+	6600 2900 5900 2900
+Wire Wire Line
+	5900 2900 5900 3300
+$Comp
+L R R2
+U 1 1 59CC4726
+P 6550 3200
+F 0 "R2" V 6630 3200 50  0000 C CNN
+F 1 "R" V 6550 3200 50  0000 C CNN
+F 2 "" V 6480 3200 50  0001 C CNN
+F 3 "" H 6550 3200 50  0001 C CNN
+	1    6550 3200
+	0    1    1    0
+$EndComp
+$Comp
+L R R1
+U 1 1 59CC47A1
+P 6200 3400
+F 0 "R1" V 6280 3400 50  0000 C CNN
+F 1 "R" V 6200 3400 50  0000 C CNN
+F 2 "" V 6130 3400 50  0001 C CNN
+F 3 "" H 6200 3400 50  0001 C CNN
+	1    6200 3400
+	0    1    1    0
+$EndComp
+Wire Wire Line
+	5700 3400 6050 3400
+Wire Wire Line
+	6350 3400 6900 3400
+Wire Wire Line
+	6900 3400 6900 3100
 $EndSCHEMATC

Commit message: Using Wemo esp8266 instead of NodeMCU
Parts:
- added R4, R5, R6: R, symbol R
- added U?: LM1084IS-3.3/NOPB, TO_SOT_Packages_SMD:TO-263-3Lead, symbol LM1084IS-3.3/NOPB
Connections:
- net labels added: +5V
- wire segments 23 -> 46
Changed lines of the file:
@@
 	-1   0    0    1
 $EndComp
-Wire Wire Line
-	4500 3500 4450 3500
-Wire Wire Line
-	4450 3500 4450 3950
-Wire Wire Line
-	4500 3400 4350 3400
-$Comp
-L GND #PWR01
+$Comp
+L GND #PWR3
 U 1 1 59CB0D77
 P 5800 3650
-F 0 "#PWR01" H 5800 3400 50  0001 C CNN
+F 0 "#PWR3" H 5800 3400 50  0001 C CNN
 F 1 "GND" H 5800 3500 50  0000 C CNN
 F 2 "" H 5800 3650 50  0001 C CNN
@@
 $EndComp
 $Comp
-L GND #PWR02
+L GND #PWR2
 U 1 1 59CB0DA4
 P 5700 2600
-F 0 "#PWR02" H 5700 2350 50  0001 C CNN
+F 0 "#PWR2" H 5700 2350 50  0001 C CNN
 F 1 "GND" H 5700 2450 50  0000 C CNN
 F 2 "" H 5700 2600 50  0001 C CNN
@@
 	-1   0    0    1
 $EndComp
-Wire Wire Line
-	5700 2800 5700 2600
-Wire Wire Line
-	5700 3500 5800 3500
-Wire Wire Line
-	5800 3500 5800 3650
-Wire Wire Line
-	6700 3200 7400 3200
-$Comp
-L +3.3V #PWR03
+$Comp
+L +3.3V #PWR1
 U 1 1 59CB1055
 P 4250 3100
-F 0 "#PWR03" H 4250 2950 50  0001 C CNN
+F 0 "#PWR1" H 4250 2950 50  0001 C CNN
 F 1 "+3.3V" H 4250 3240 50  0000 C CNN
 F 2 "" H 4250 3100 50  0001 C CNN
@@
 	0    -1   -1   0
 $EndComp
-Wire Wire Line
-	4500 3100 4250 3100
-Wire Wire Line
-	4350 3400 4350 3950
-$Comp
-L GND #PWR04
+$Comp
+L GND #PWR5
 U 1 1 59CB1286
 P 7150 3700
-F 0 "#PWR04" H 7150 3450 50  0001 C CNN
+F 0 "#PWR5" H 7150 3450 50  0001 C CNN
 F 1 "GND" H 7150 3550 50  0000 C CNN
 F 2 "" H 7150 3700 50  0001 C CNN
@@
 	0    1    1    0
 $EndComp
-Wire Wire Line
-	7400 3700 7150 3700
-$Comp
-L +3.3V #PWR05
+$Comp
+L +3.3V #PWR6
 U 1 1 59CB12BC
 P 8500 3800
-F 0 "#PWR05" H 8500 3650 50  0001 C CNN
+F 0 "#PWR6" H 8500 3650 50  0001 C CNN
 F 1 "+3.3V" H 8500 3940 50  0000 C CNN
 F 2 "" H 8500 3800 50  0001 C CNN
@@
 	0    1    1    0
 $EndComp
-Wire Wire Line
-	8300 3800 8500 3800
 Text Label 7100 2900 0    60   ~ 0
 MOSI
-Wire Wire Line
-	7400 3100 6900 3100
 Text Label 7100 3100 0    60   ~ 0
 MISO
 $Comp
-L +3.3V #PWR06
+L +3.3V #PWR4
 U 1 1 59CB148A
 P 7100 3400
-F 0 "#PWR06" H 7100 3250 50  0001 C CNN
+F 0 "#PWR4" H 7100 3250 50  0001 C CNN
 F 1 "+3.3V" H 7100 3540 50  0000 C CNN
 F 2 "" H 7100 3400 50  0001 C CNN
@@
 	0    -1   -1   0
 $EndComp
-Wire Wire Line
-	7400 3400 7100 3400
 Text Label 7150 3000 0    60   ~ 0
 CS
@@
 	0    1    1    0
 $EndComp
-Wire Wire Line
-	7150 1700 3300 1700
-Wire Wire Line
-	3300 1700 3300 550
-Wire Wire Line
-	7400 2900 6900 2900
-Wire Wire Line
-	5700 3300 5900 3300
-Wire Wire Line
-	5700 3200 6400 3200
-Wire Wire Line
-	6600 2900 5900 2900
-Wire Wire Line
-	5900 2900 5900 3300
 $Comp
 L R R2
@@
 $EndComp
 Wire Wire Line
+	4500 3500 4450 3500
+Wire Wire Line
+	4450 3500 4450 3950
+Wire Wire Line
+	4500 3400 4350 3400
+Wire Wire Line
+	5700 2800 5700 2600
+Wire Wire Line
+	5700 3500 5800 3500
+Wire Wire Line
+	5800 3500 5800 3650
+Wire Wire Line
+	6700 3200 7400 3200
+Wire Wire Line
+	4500 3100 4250 3100
+Wire Wire Line
+	4350 3400 4350 3950
+Wire Wire Line
+	7400 3700 7150 3700
+Wire Wire Line
+	8300 3800 8500 3800
+Wire Wire Line
+	7400 3100 6900 3100
+Wire Wire Line
+	7400 3400 7100 3400
+Wire Wire Line
+	7400 2900 6900 2900
+Wire Wire Line
+	5700 3300 5900 3300
+Wire Wire Line
+	5700 3200 6400 3200
+Wire Wire Line
+	6600 2900 5900 2900
+Wire Wire Line
+	5900 2900 5900 3300
+Wire Wire Line
 	5700 3400 6050 3400
 Wire Wire Line
@@
 Wire Wire Line
 	6900 3400 6900 3100
+$Comp
+L R R4
+U 1 1 59CF0F92
+P 6300 3050
+F 0 "R4" V 6380 3050 50  0000 C CNN
+F 1 "R" V 6300 3050 50  0000 C CNN
+F 2 "" V 6230 3050 50  0001 C CNN
+F 3 "" H 6300 3050 50  0001 C CNN
+	1    6300 3050
+	0    1    1    0
+$EndComp
+Wire Wire Line
+	7400 3000 6850 3000
+Wire Wire Line
+	6850 3000 6850 3050
+Wire Wire Line
+	6850 3050 6450 3050
+Wire Wire Line
+	6150 3050 6100 3050
+Wire Wire Line
+	6100 3050 6100 3100
+Wire Wire Line
+	6100 3100 5700 3100
+$Comp
+L R R6
+U 1 1 59CF1001
+P 6400 2700
+F 0 "R6" V 6480 2700 50  0000 C CNN
+F 1 "R" V 6400 2700 50  0000 C CNN
+F 2 "" V 6330 2700 50  0001 C CNN
+F 3 "" H 6400 2700 50  0001 C CNN
+	1    6400 2700
+	0    1    1    0
+$EndComp
+Wire Wire Line
+	8450 2050 8450 2700
+Wire Wire Line
+	8450 2050 7000 2050
+Wire Wire Line
+	7000 2050 7000 2700
+Wire Wire Line
+	7000 2700 6550 2700
+Wire Wire Line
+	6250 2700 5850 2700
+Wire Wire Line
+	5850 2700 5850 3000
+Wire Wire Line
+	5850 3000 5700 3000
+$Comp
+L R R5
+U 1 1 59CF1A56
+P 6400 2450
+F 0 "R5" V 6480 2450 50  0000 C CNN
+F 1 "R" V 6400 2450 50  0000 C CNN
+F 2 "" V 6330 2450 50  0001 C CNN
+F 3 "" H 6400 2450 50  0001 C CNN
+	1    6400 2450
+	0    1    1    0
+$EndComp
+Wire Wire Line
+	4500 3000 4250 3000
+Wire Wire Line
+	4250 3000 4250 2300
+Wire Wire Line
+	4250 2300 6250 2300
+Wire Wire Line
+	6250 2300 6250 2450
+Wire Wire Line
+	6550 2450 6550 1900
+Wire Wire Line
+	6550 1900 8600 1900
+Wire Wire Line
+	8600 1900 8600 2800
+Wire Wire Line
+	8600 2800 8300 2800
+Wire Wire Line
+	8450 2700 8300 2700
+$Comp
+L LM1084IS-3.3/NOPB U?
+U 1 1 59D2FBBD
+P 6450 4500
+F 0 "U?" H 6650 4300 50  0000 C CNN
+F 1 "LM1084IS-3.3/NOPB" H 6150 4700 50  0000 L CNN
+F 2 "TO_SOT_Packages_SMD:TO-263-3Lead" H 6450 4600 50  0001 C CIN
+F 3 "" H 6450 4500 50  0001 C CNN
+	1    6450 4500
+	-1   0    0    1
+$EndComp
+$Comp
+L GND #PWR?
+U 1 1 59D2FC8A
+P 6450 4150
+F 0 "#PWR?" H 6450 3900 50  0001 C CNN
+F 1 "GND" H 6450 4000 50  0000 C CNN
+F 2 "" H 6450 4150 50  0001 C CNN
+F 3 "" H 6450 4150 50  0001 C CNN
+	1    6450 4150
+	-1   0    0    1
+$EndComp
+Wire Wire Line
+	6450 4150 6450 4250
+$Comp
+L +3.3V #PWR?
+U 1 1 59D2FCFE
+P 5800 4550
+F 0 "#PWR?" H 5800 4400 50  0001 C CNN
+F 1 "+3.3V" H 5800 4690 50  0000 C CNN
+F 2 "" H 5800 4550 50  0001 C CNN
+F 3 "" H 5800 4550 50  0001 C CNN
+	1    5800 4550
+	0    -1   -1   0
+$EndComp
+Wire Wire Line
+	5800 4550 6050 4550
+$Comp
+L +5V #PWR?
+U 1 1 59D2FD9A
+P 7050 4550
+F 0 "#PWR?" H 7050 4400 50  0001 C CNN
+F 1 "+5V" H 7050 4690 50  0000 C CNN
+F 2 "" H 7050 4550 50  0001 C CNN
+F 3 "" H 7050 4550 50  0001 C CNN
+	1    7050 4550
+	0    1    1    0
+$EndComp
+Wire Wire Line
+	6850 4550 7050 4550
 $EndSCHEMATC

Commit message: Finalized schematic, first run at board layout.
Parts:
- removed U2: NodeMCU_Amica_R2, symbol NodeMCU_Amica_R2
- added U3: WeMos_mini, DisasterRadio:D1_mini_Hat, symbol WeMos_mini
- AE1: footprint (none) -> Connectors:SMA_SMD_Jack_Straight
- R1: renamed from R5; value R -> 0k; footprint (none) -> Resistors_SMD:R_0805
- R2: renamed from R6; value R -> 0k; footprint (none) -> Resistors_SMD:R_0805
- R3, R4: value R -> 0k; footprint (none) -> Resistors_SMD:R_0805
- R5: renamed from R2; value R -> 0k; footprint (none) -> Resistors_SMD:R_0805
- R6: renamed from R1; value R -> 0k; footprint (none) -> Resistors_SMD:R_0805
- gave numbers to parts that had none: 1
Connections:
- net labels added: SCK, SS
- net labels removed: CS
- wire segments 46 -> 50
- no-connect marks 0 -> 12
Other:
- moved on the sheet: R1, R2, R3, R4, R5, R6

Commit message: Relayed out board.
Parts:
- removed U2: LM1084IS-3.3/NOPB, TO_SOT_Packages_SMD:TO-263-3Lead, symbol LM1084IS-3.3/NOPB
- added C1, C2: 10u, symbol C
- added U2: LM1117-3.3, symbol LM1117-3.3
Connections:
- wire segments 50 -> 54
Changed lines of the file:
@@
 $EndComp
 $Comp
-L GND #PWR01
+L GND #PWR3
 U 1 1 59CB0D77
 P 5800 3650
-F 0 "#PWR01" H 5800 3400 50  0001 C CNN
+F 0 "#PWR3" H 5800 3400 50  0001 C CNN
 F 1 "GND" H 5800 3500 50  0000 C CNN
 F 2 "" H 5800 3650 50  0001 C CNN
@@
 $EndComp
 $Comp
-L GND #PWR02
+L GND #PWR2
 U 1 1 59CB0DA4
 P 5700 2700
-F 0 "#PWR02" H 5700 2450 50  0001 C CNN
+F 0 "#PWR2" H 5700 2450 50  0001 C CNN
 F 1 "GND" H 5700 2550 50  0000 C CNN
 F 2 "" H 5700 2700 50  0001 C CNN
@@
 $EndComp
 $Comp
-L +3.3V #PWR03
+L +3.3V #PWR1
 U 1 1 59CB1055
 P 4250 3100
-F 0 "#PWR03" H 4250 2950 50  0001 C CNN
+F 0 "#PWR1" H 4250 2950 50  0001 C CNN
 F 1 "+3.3V" H 4250 3240 50  0000 C CNN
 F 2 "" H 4250 3100 50  0001 C CNN
@@
 	4500 3000 4250 3000
 $Comp
-L LM1084IS-3.3/NOPB U2
-U 1 1 59D2FBBD
-P 6450 4500
-F 0 "U2" H 6650 4300 50  0000 C CNN
-F 1 "LM1084IS-3.3/NOPB" H 6150 4700 50  0000 L CNN
-F 2 "TO_SOT_Packages_SMD:TO-263-3Lead" H 6450 4600 50  0001 C CIN
-F 3 "" H 6450 4500 50  0001 C CNN
-	1    6450 4500
-	-1   0    0    1
-$EndComp
-$Comp
-L GND #PWR04
+L GND #PWR7
 U 1 1 59D2FC8A
-P 6450 4150
-F 0 "#PWR04" H 6450 3900 50  0001 C CNN
-F 1 "GND" H 6450 4000 50  0000 C CNN
-F 2 "" H 6450 4150 50  0001 C CNN
-F 3 "" H 6450 4150 50  0001 C CNN
-	1    6450 4150
-	-1   0    0    1
-$EndComp
-Wire Wire Line
-	6450 4150 6450 4250
-$Comp
-L +3.3V #PWR05
+P 7800 5150
+F 0 "#PWR7" H 7800 4900 50  0001 C CNN
+F 1 "GND" H 7800 5000 50  0000 C CNN
+F 2 "" H 7800 5150 50  0001 C CNN
+F 3 "" H 7800 5150 50  0001 C CNN
+	1    7800 5150
+	1    0    0    -1
+$EndComp
+$Comp
+L +3.3V #PWR8
 U 1 1 59D2FCFE
-P 5800 4550
-F 0 "#PWR05" H 5800 4400 50  0001 C CNN
-F 1 "+3.3V" H 5800 4690 50  0000 C CNN
-F 2 "" H 5800 4550 50  0001 C CNN
-F 3 "" H 5800 4550 50  0001 C CNN
-	1    5800 4550
-	0    -1   -1   0
-$EndComp
-Wire Wire Line
-	5800 4550 6050 4550
-$Comp
-L +5V #PWR06
+P 8600 4550
+F 0 "#PWR8" H 8600 4400 50  0001 C CNN
+F 1 "+3.3V" H 8600 4690 50  0000 C CNN
+F 2 "" H 8600 4550 50  0001 C CNN
+F 3 "" H 8600 4550 50  0001 C CNN
+	1    8600 4550
+	0    1    1    0
+$EndComp
+$Comp
+L +5V #PWR4
 U 1 1 59D2FD9A
 P 7050 4550
-F 0 "#PWR06" H 7050 4400 50  0001 C CNN
+F 0 "#PWR4" H 7050 4400 50  0001 C CNN
 F 1 "+5V" H 7050 4690 50  0000 C CNN
 F 2 "" H 7050 4550 50  0001 C CNN
 F 3 "" H 7050 4550 50  0001 C CNN
 	1    7050 4550
-	0    1    1    0
-$EndComp
-Wire Wire Line
-	6850 4550 7050 4550
+	0    -1   -1   0
+$EndComp
 Wire Wire Line
 	6050 3400 6050 3650
@@
 $EndComp
 $Comp
-L +5V #PWR07
+L +5V #PWR6
 U 1 1 59DAD071
 P 7700 2400
-F 0 "#PWR07" H 7700 2250 50  0001 C CNN
+F 0 "#PWR6" H 7700 2250 50  0001 C CNN
 F 1 "+5V" H 7700 2540 50  0000 C CNN
 F 2 "" H 7700 2400 50  0001 C CNN
@@
 $EndComp
 $Comp
-L GND #PWR08
+L GND #PWR5
 U 1 1 59DAD0A3
 P 7500 2400
-F 0 "#PWR08" H 7500 2150 50  0001 C CNN
+F 0 "#PWR5" H 7500 2150 50  0001 C CNN
 F 1 "GND" H 7500 2250 50  0000 C CNN
 F 2 "" H 7500 2400 50  0001 C CNN
@@
 $EndComp
 $Comp
-L +3.3V #PWR09
+L +3.3V #PWR9
 U 1 1 59DAD0D5
 P 9000 2400
-F 0 "#PWR09" H 9000 2250 50  0001 C CNN
+F 0 "#PWR9" H 9000 2250 50  0001 C CNN
 F 1 "+3.3V" H 9000 2540 50  0000 C CNN
 F 2 "" H 9000 2400 50  0001 C CNN
@@
 NoConn ~ 4500 2900
 NoConn ~ 4500 2800
+$Comp
+L LM1117-3.3 U2
+U 1 1 59DDA3AE
+P 7800 4550
+F 0 "U2" H 7900 4300 50  0000 C CNN
+F 1 "LM1117-3.3" H 7800 4800 50  0000 C CNN
+F 2 "" H 7800 4550 50  0001 C CNN
+F 3 "" H 7800 4550 50  0001 C CNN
+	1    7800 4550
+	1    0    0    -1
+$EndComp
+$Comp
+L C C2
+U 1 1 59DDA417
+P 8350 4750
+F 0 "C2" H 8375 4850 50  0000 L CNN
+F 1 "10u" H 8375 4650 50  0000 L CNN
+F 2 "" H 8388 4600 50  0001 C CNN
+F 3 "" H 8350 4750 50  0001 C CNN
+	1    8350 4750
+	-1   0    0    1
+$EndComp
+$Comp
+L C C1
+U 1 1 59DDA458
+P 7300 4850
+F 0 "C1" H 7325 4950 50  0000 L CNN
+F 1 "10u" H 7325 4750 50  0000 L CNN
+F 2 "" H 7338 4700 50  0001 C CNN
+F 3 "" H 7300 4850 50  0001 C CNN
+	1    7300 4850
+	-1   0    0    1
+$EndComp
+Wire Wire Line
+	8100 4550 8600 4550
+Wire Wire Line
+	7050 4550 7500 4550
+Wire Wire Line
+	7800 4850 7800 5150
+Wire Wire Line
+	7300 4700 7300 4550
+Connection ~ 7300 4550
+Wire Wire Line
+	8350 4550 8350 4600
+Connection ~ 8350 4550
+Wire Wire Line
+	7300 5000 8350 5000
+Wire Wire Line
+	8350 5000 8350 4900
+Connection ~ 7800 5000
 $EndSCHEMATC
