File: lora_nodemcu.kicad_pcb (KiCad board)
At the start: 4 copper layers, 25.8 x 32.9 mm, 17 parts, among them U1 RFM95, U2 LM1117-3.3, U3 WeMos_mini

Commit message: updated bottom silkscreen and added fp-lib-table
Other:
- board text added: "0.1uF"
- board text added: "10uF"
- board text added: "Disaster Radio V0.2 180109"
- board text added: "JUMPER"
- board text added: "https://disaster.radio/"
Changed lines of the file:
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@@
   (general
     (thickness 1.2)
-    (drawings 16)
+    (drawings 31)
     (tracks 157)
     (zones 0)
@@
     (pad_to_mask_clearance 0.2)
     (aux_axis_origin 0 0)
-    (visible_elements FFFEFFBF)
+    (visible_elements FFFFFFFF)
     (pcbplotparams
       (layerselection 0x010f0_ffffffff)
@@
       (effects (font (size 1 1) (thickness 0.15)))
     )
-    (fp_line (start -6.35 3.81) (end -6.35 -10.16) (layer B.SilkS) (width 0.15))
-    (fp_line (start -6.35 -10.16) (end 6.35 -10.16) (layer B.SilkS) (width 0.15))
-    (fp_line (start 6.35 -10.16) (end 6.35 3.81) (layer B.SilkS) (width 0.15))
-    (fp_line (start 6.35 3.81) (end -6.35 3.81) (layer B.SilkS) (width 0.15))
-    (fp_line (start -8.89 5.08) (end 8.89 5.08) (layer B.SilkS) (width 0.15))
-    (fp_line (start 8.89 5.08) (end 8.89 -17.78) (layer B.SilkS) (width 0.15))
-    (fp_line (start 8.89 -17.78) (end -8.89 -17.78) (layer B.SilkS) (width 0.15))
-    (fp_line (start -8.89 -17.78) (end -8.89 5.08) (layer B.SilkS) (width 0.15))
     (pad 8 thru_hole circle (at -11.43 -10.16) (size 1.8 1.8) (drill 1.016) (layers *.Cu *.Mask F.SilkS)
       (net 21 "Net-(U3-Pad8)"))
@@
     (tags "capacitor 0805")
     (attr smd)
-    (fp_text reference C5 (at 0 1.75) (layer B.SilkS)
+    (fp_text reference C5 (at -3.45 0.05) (layer B.SilkS)
       (effects (font (size 1 1) (thickness 0.15)) (justify mirror))
     )
@@
     (tags "capacitor 0805")
     (attr smd)
-    (fp_text reference C4 (at 0 1.75 270) (layer B.SilkS)
+    (fp_text reference C4 (at -0.25 -2.1 270) (layer B.SilkS)
       (effects (font (size 1 1) (thickness 0.15)) (justify mirror))
     )
@@
     (tags "resistor 0805")
     (attr smd)
-    (fp_text reference L1 (at 0 2.1) (layer B.SilkS)
+    (fp_text reference L1 (at 0 -1.8) (layer B.SilkS)
       (effects (font (size 1 1) (thickness 0.15)) (justify mirror))
     )
@@
     (tags "capacitor 0805")
     (attr smd)
-    (fp_text reference C1 (at 0 1.75 270) (layer B.SilkS)
+    (fp_text reference C1 (at 3.4 -0.15 270) (layer B.SilkS)
       (effects (font (size 1 1) (thickness 0.15)) (justify mirror))
     )
@@
     (tags "capacitor 0805")
     (attr smd)
-    (fp_text reference C2 (at 0 1.75 270) (layer B.SilkS)
+    (fp_text reference C2 (at 3.5 0 270) (layer B.SilkS)
       (effects (font (size 1 1) (thickness 0.15)) (justify mirror))
     )
@@
     (tags "resistor 0805")
     (attr smd)
-    (fp_text reference R1 (at 0 1.7) (layer B.SilkS)
+    (fp_text reference R1 (at 3.55 0) (layer B.SilkS)
       (effects (font (size 1 1) (thickness 0.15)) (justify mirror))
     )
@@
     (tags "resistor 0805")
     (attr smd)
-    (fp_text reference R2 (at 0 1.7) (layer B.SilkS)
+    (fp_text reference R2 (at 3.35 -0.1) (layer B.SilkS)
       (effects (font (size 1 1) (thickness 0.15)) (justify mirror))
     )
@@
     (tags "resistor 0805")
     (attr smd)
-    (fp_text reference R3 (at 0 1.7 180) (layer B.SilkS)
+    (fp_text reference R3 (at 3.45 -0.1 180) (layer B.SilkS)
       (effects (font (size 1 1) (thickness 0.15)) (justify mirror))
     )
@@
     (tags "resistor 0805")
     (attr smd)
-    (fp_text reference R4 (at 0 1.7 180) (layer B.SilkS)
+    (fp_text reference R4 (at 3.4 -0.05 180) (layer B.SilkS)
       (effects (font (size 1 1) (thickness 0.15)) (justify mirror))
     )
@@
     (tags "resistor 0805")
     (attr smd)
-    (fp_text reference R5 (at 0 1.7 180) (layer B.SilkS)
+    (fp_text reference R5 (at 3.55 0 180) (layer B.SilkS)
       (effects (font (size 1 1) (thickness 0.15)) (justify mirror))
     )
@@
     (tags "resistor 0805")
     (attr smd)
-    (fp_text reference R6 (at 0 1.7 180) (layer B.SilkS)
+    (fp_text reference R6 (at 3.8 -0.05 180) (layer B.SilkS)
       (effects (font (size 1 1) (thickness 0.15)) (justify mirror))
     )
@@
     )
   )
+  (gr_text 0.1uF (at 140.7 93.4) (layer B.SilkS)
+    (effects (font (size 0.5 0.5) (thickness 0.1)) (justify mirror))
+  )
+  (gr_text 10uF (at 156.95 102.7 90) (layer B.SilkS)
+    (effects (font (size 0.5 0.5) (thickness 0.1)) (justify mirror))
+  )
+  (gr_text 10uF (at 152.45 102.8 90) (layer B.SilkS)
+    (effects (font (size 0.5 0.5) (thickness 0.1)) (justify mirror))
+  )
+  (gr_text JUMPER (at 156.75 99.7) (layer B.SilkS)
+    (effects (font (size 0.5 0.5) (thickness 0.1)) (justify mirror))
+  )
+  (gr_text 0.1uF (at 151.1 99.65) (layer B.SilkS)
+    (effects (font (size 0.5 0.5) (thickness 0.1)) (justify mirror))
+  )
+  (gr_text JUMPER (at 148.25 96.6 90) (layer B.SilkS)
+    (effects (font (size 0.5 0.5) (thickness 0.1)) (justify mirror))
+  )
+  (gr_text 0.1uF (at 153.8 95.35) (layer B.SilkS)
+    (effects (font (size 0.5 0.5) (thickness 0.1)) (justify mirror))
+  )
+  (gr_text JUMPER (at 154.45 90) (layer B.SilkS)
+    (effects (font (size 0.5 0.5) (thickness 0.1)) (justify mirror))
+  )
+  (gr_text JUMPER (at 154.4 87.15) (layer B.SilkS)
+    (effects (font (size 0.5 0.5) (thickness 0.1)) (justify mirror))
+  )
+  (gr_text JUMPER (at 154.45 84.2) (layer B.SilkS)
+    (effects (font (size 0.5 0.5) (thickness 0.1)) (justify mirror))
+  )
+  (gr_text JUMPER (at 154.5 80.8) (layer B.SilkS)
+    (effects (font (size 0.5 0.5) (thickness 0.1)) (justify mirror))
+  )
+  (gr_text JUMPER (at 144.8 83.4) (layer B.SilkS)
+    (effects (font (size 0.5 0.5) (thickness 0.1)) (justify mirror))
+  )
+  (gr_text JUMPER (at 144.75 80.55) (layer B.SilkS)
+    (effects (font (size 0.5 0.5) (thickness 0.1)) (justify mirror))
+  )
+  (gr_text https://disaster.radio/ (at 147.8 77.3) (layer B.SilkS)
+    (effects (font (size 0.5 0.5) (thickness 0.1)) (justify mirror))
+  )
+  (gr_text "Disaster Radio V0.2 180109" (at 147.85 76.25) (layer B.SilkS)
+    (effects (font (size 0.5 0.5) (thickness 0.1)) (justify mirror))
+  )
   (gr_text 5V (at 139.15 94.75) (layer F.SilkS)
