File: hardware/board_v3/lora_nodemcu.sch (KiCad schematic (older format))
At the start: 23 parts, among them U1 RFM95, U3 WeMos_mini

Commit message: Just about finished board v3 schematic
Parts:
- added C? (x2): 0.1uF, symbol Device:C_Small
- added J?: LiPo 18650, symbol Connector_Generic:Conn_01x02
- added J?: Solar Panel, symbol Connector_Generic:Conn_01x02
- added J?: ESP_PRGM, symbol Connector_Generic:Conn_01x04
- added J?: RESET_BUTTON, symbol Connector_Generic:Conn_01x02
- added J?: RGB_LED, symbol Connector_Generic:Conn_01x04
- added JP?: CS, symbol Jumper:Jumper_2_Bridged
- added JP?: RST, symbol Jumper:Jumper_2_Bridged
- added JP?: D1, symbol Jumper:Jumper_2_Bridged
- added L?: JUMPER, symbol Device:L_Core_Ferrite_Small
- added R? (x5): 10K, symbol Device:R_Small
- added SW?: SW_SPST, symbol Switch:SW_SPST
- added U?: CN3791_module, symbol disaster_radio:CN3791_module
- JP?: value JUMPER -> MISO
- JP?: value JUMPER -> MOSI
- JP?: value JUMPER -> CLK
Connections:
- net labels added: +BATT, SPI_CLK, SPI_MISO, SPI_MOSI
- wire segments 62 -> 167
Other:
- moved on the sheet: AE?, C?, JP?, U?

Commit message: updates schematic, associates all footprints, beginning pcb layout
Parts:
- removed AE1: Antenna_Shield, Connectors_Molex:Molex_SMA_Jack_Edge_Mount, symbol lora_nodemcu-rescue:Antenna_Shield-device
- removed C3: C_Small, Capacitors_SMD:C_0805_HandSoldering, symbol lora_nodemcu-rescue:C_Small-device
- removed C4, C5: C_decoupling, Capacitors_SMD:C_0805_HandSoldering, symbol lora_nodemcu-rescue:C_Small-device
- removed L1: L_Core_Ferrite_Small, Inductors_SMD:L_0805_HandSoldering, symbol lora_nodemcu-rescue:L_Core_Ferrite_Small-device
- removed L2: L_Core_Ferrite, Inductors_SMD:L_0805_HandSoldering, symbol lora_nodemcu-rescue:L_Core_Ferrite_Small-device
- removed R1, R2, R3, R4, R5, R6: 0k, Resistors_SMD:R_0805_HandSoldering, symbol lora_nodemcu-rescue:R-device
- removed R?: 10K, symbol Device:R_Small
- removed U1: RFM95, DisasterRadio:RFM95, symbol rfm95:RFM95
- removed U3: WeMos_mini, DisasterRadio:D1_mini_board, symbol lora_nodemcu-rescue:WeMos_mini-RESCUE-lora_nodemcu
- added J6: RF_Shield_ESP-07S, RF_Shielding:Wuerth_36103305_30x30mm, symbol Device:RF_Shield_One_Piece
- added J7: RF_Shield_RFM95, RF_Shielding:Wuerth_36103305_30x30mm, symbol Device:RF_Shield_One_Piece
- added JP1: SOLAR_TP, Jumper:SolderJumper-2_P1.3mm_Bridged_Pad1.0x1.5mm, symbol Jumper:Jumper_2_Bridged
- added JP2: LiPo_TP, Jumper:SolderJumper-2_P1.3mm_Bridged_Pad1.0x1.5mm, symbol Jumper:Jumper_2_Bridged
- added JP3: PRGM_SELECT, Connector_PinHeader_2.54mm:PinHeader_1x03_P2.54mm_Vertical, symbol Device:Jumper_NC_Dual
- added L2: JUMPER, Inductor_SMD:L_0805_2012Metric_Pad1.15x1.50mm_HandSolder, symbol Device:L_Core_Ferrite_Small
- added Q1, Q2, Q3: 2N3904, Package_TO_SOT_SMD:SOT-23_Handsoldering, symbol Transistor_BJT:2N3904
- added R10: 1K, Resistor_SMD:R_0805_2012Metric_Pad1.15x1.50mm_HandSolder, symbol Device:R_Small
- added R11, R13, R3, R5, R8, R9: 10K, Resistor_SMD:R_0805_2012Metric_Pad1.15x1.50mm_HandSolder, symbol Device:R_Small
- added R12: 470, Resistor_SMD:R_0805_2012Metric_Pad1.15x1.50mm_HandSolder, symbol Device:R_Small
- added R14: 330, Resistor_SMD:R_0805_2012Metric_Pad1.15x1.50mm_HandSolder, symbol Device:R_Small
- added R2: 47K, Resistor_SMD:R_0805_2012Metric_Pad1.15x1.50mm_HandSolder, symbol Device:R_Small
- AE1: renamed from AE?; value Antenna_Shield -> RFM95_Antenna; footprint Connectors_Molex:Molex_SMA_Jack_Edge_Mount -> Connector_Coaxial:U.FL_Hirose_U.FL-R-SMT-1_Vertical
- C1, C4: renamed from C?; footprint (none) -> Capacitor_SMD:C_0805_2012Metric_Pad1.15x1.50mm_HandSolder
- C2, C3: renamed from C?; value C_Small -> 10uF; footprint (none) -> Capacitor_SMD:C_0805_2012Metric_Pad1.15x1.50mm_HandSolder
- J1, J3: renamed from J?; footprint (none) -> Connector_Phoenix_MC:PhoenixContact_MCV_1,5_2-G-5.08_1x02_P5.08mm_Vertical
- J2: renamed from J?; footprint (none) -> Battery:BatteryHolder_MPD_BH-18650-PC2
- J4: renamed from J?; footprint (none) -> Connector_PinHeader_2.54mm:PinHeader_1x04_P2.54mm_Vertical
- J5: renamed from J?; footprint (none) -> Connector_Phoenix_MC:PhoenixContact_MCV_1,5_4-G-5.08_1x04_P5.08mm_Vertical
- JP4, JP5, JP6, JP7, JP8, JP9: renamed from JP?; footprint (none) -> Jumper:SolderJumper-2_P1.3mm_Bridged_Pad1.0x1.5mm
- L1: renamed from L?; footprint (none) -> Inductor_SMD:L_0805_2012Metric_Pad1.15x1.50mm_HandSolder
- R1, R4, R6, R7: renamed from R?; footprint (none) -> Resistor_SMD:R_0805_2012Metric_Pad1.15x1.50mm_HandSolder
- SW1: renamed from SW?; footprint (none) -> Connector_Phoenix_MC:PhoenixContact_MCV_1,5_2-G-5.08_1x02_P5.08mm_Vertical
- U1: renamed from U?; footprint (none) -> disaster_radio:CN3791_module
- U2: renamed from U?; footprint (none) -> ESP8266:ESP-07S
- U3: renamed from U?; footprint (none) -> Package_TO_SOT_SMD:SOT-223-3_TabPin2
- U4: renamed from U?; footprint (none) -> disaster_radio:RFM95
Connections:
- net labels added: BLUE, GREEN, RED
- net labels removed: +5V, 50Ohm, MISO, MOSI, RF95_3V3, SCK, SS, wemos_5V
- wire segments 167 -> 157
- no-connect marks 12 -> 0
Other:
- note removed: "OLD SCHEMATIC TO BE REMOVED"
- moved on the sheet: AE1, C1, C2, C3, C4, J1, J2, J3, J4, J5, JP4, JP5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

Commit message: places all components in just about final location
Parts:
- added JP10: MPPT_TP, Jumper:SolderJumper-2_P1.3mm_Bridged_Pad1.0x1.5mm, symbol Jumper:Jumper_2_Bridged
- added R? (x2): 10K, Resistor_SMD:R_0805_2012Metric_Pad1.15x1.50mm_HandSolder, symbol Device:R_Small
Connections:
- net +BATT: now also JP10.1 (A); no longer U1.3 (Battery+)
- net at Q3.2 (B), R13.2: now also R?.1; no longer U2.13 (GPIO4)
- net at Q2.2 (B), R11.2: now also R?.1; no longer U2.14 (GPIO5)
- new net: R?.2, U2.13 (GPIO4)
- new net: R?.2, U2.14 (GPIO5)
- new net: JP10.2 (B), U1.3 (Battery+)
Changed lines of the file:
@@
 	5950 2300 5950 3450
-Wire Wire Line
-	5950 3450 4950 3450
 Wire Wire Line
 	4350 3850 4350 3550
@@
 Wire Wire Line
 	4700 3450 4850 3450
-Connection ~ 4950 3450
 $Comp
 L Jumper:Jumper_2_Bridged JP1
@@
 	11700 4550 11700 4900
 Wire Wire Line
-	11700 5500 7450 5500
-Wire Wire Line
 	7450 5500 7450 6300
 Wire Wire Line
@@
 Wire Wire Line
 	11050 4550 11050 4950
-Wire Wire Line
-	11050 5350 7350 5350
 Wire Wire Line
 	7350 5350 7350 6200
@@
 	1    0    0    -1
 $EndComp
+$Comp
+L Jumper:Jumper_2_Bridged JP10
+U 1 1 5AADE3CF
+P 5450 3450
+F 0 "JP10" H 5450 3645 50  0000 C CNN
+F 1 "MPPT_TP" H 5450 3554 50  0000 C CNN
+F 2 "Jumper:SolderJumper-2_P1.3mm_Bridged_Pad1.0x1.5mm" H 5450 3450 50  0001 C CNN
+F 3 "~" H 5450 3450 50  0001 C CNN
+	1    5450 3450
+	1    0    0    -1
+$EndComp
+Wire Wire Line
+	5250 3450 4950 3450
+Connection ~ 4950 3450
+Wire Wire Line
+	5650 3450 5950 3450
+$Comp
+L Device:R_Small R?
+U 1 1 5AAECE0B
+P 8300 5350
+F 0 "R?" V 8400 5300 50  0000 L CNN
+F 1 "10K" V 8200 5300 50  0000 L CNN
+F 2 "Resistor_SMD:R_0805_2012Metric_Pad1.15x1.50mm_HandSolder" H 8300 5350 50  0001 C CNN
+F 3 "~" H 8300 5350 50  0001 C CNN
+	1    8300 5350
+	0    1    -1   0
+$EndComp
+$Comp
+L Device:R_Small R?
+U 1 1 5AAED216
+P 8650 5500
+F 0 "R?" V 8750 5450 50  0000 L CNN
+F 1 "10K" V 8550 5450 50  0000 L CNN
+F 2 "Resistor_SMD:R_0805_2012Metric_Pad1.15x1.50mm_HandSolder" H 8650 5500 50  0001 C CNN
+F 3 "~" H 8650 5500 50  0001 C CNN
+	1    8650 5500
+	0    1    -1   0
+$EndComp
+Wire Wire Line
+	8550 5500 7450 5500
+Wire Wire Line
+	8200 5350 7350 5350
+Wire Wire Line
+	11050 5350 8400 5350
+Wire Wire Line
+	11700 5500 8750 5500
 $EndSCHEMATC
